Commit message: [feat] mbot_gazeob at last

File: mbot_gazebo/urdf/sensor/kinect.xacro (robot description, xacro)
@@ -20,4 +20,10 @@
       </collision>
     </link>
+    <joint name="kinect_optical_joint" type="fixed">
+        <origin xyz="0 0 0" rpy="-1.5708 0 -1.5708"/>
+        <parent link="kinect_link"/>
+        <child link="kinect_frame_optical"/>
+    </joint>
+    <link name="kinect_frame_optical"/>
     <gazebo reference="kinect_link">
         <sensor type="depth" name="kinect">
@@ -45,5 +51,5 @@
                 <cameraInfoTopicName>rgb/camera_info</cameraInfoTopicName>
                 <depthImageCameraInfoTopicName>depth/camera_info</depthImageCameraInfoTopicName>
-                <frameName>kinect_link</frameName>
+                <frameName>kinect_frame_optical</frameName>
                 <baseline>0.1</baseline>
                 <distortion_k1>0.0</distortion_k1>
