Commit message: [fix] up it

File: robot_hunt_maze/urdf/mbot_base.xacro (robot description, xacro)
@@ -214,5 +214,6 @@
   <xacro:robot_base />
   <xacro:include filename="$(find robot_hunt_maze)/urdf/sensor/camera.xacro" />
-  <xacro:usb_camera joint_x="${camera_joint_x}" joint_y="${camera_joint_y}" joint_z="${camera_joint_z}"/>
+  <xacro:usb_camera prefix="front"  reflect="1" turn="0" />
+  <xacro:usb_camera prefix="back"  reflect="-1" turn="${M_PI}"/>
   <xacro:include filename="$(find robot_hunt_maze)/urdf/sensor/laser.xacro" />
   <xacro:laser joint_x="${laser_joint_x}" joint_y="${laser_joint_y}" joint_z="${laser_joint_z}"/>

File: robot_hunt_maze/urdf/sensor/camera.xacro (robot description, xacro)
@@ -1,11 +1,11 @@
 <?xml version="1.0" ?>
-<robot name="mbot" xmlns:xacro="http://www.ros.org/wiki/xacro">
-  <xacro:macro name="usb_camera" params="joint_x joint_y joint_z">
-    <joint name="camera_joint" type="fixed">
-      <origin xyz="${joint_x} ${joint_y} ${joint_z}" rpy="0 0 0" />
+<robot name="camera" xmlns:xacro="http://www.ros.org/wiki/xacro">
+  <xacro:macro name="usb_camera" params="prefix reflect turn">
+    <joint name="${prefix}_camera_joint" type="fixed">
+      <origin xyz="${reflect*camera_joint_x} ${camera_joint_y} ${camera_joint_z}" rpy="0 0 ${turn}" />
       <parent link="base_link"/>
-      <child link="camera_link" />
+      <child link="${prefix}_camera_link" />
     </joint>
-    <link name="camera_link">
+    <link name="${prefix}_camera_link">
       <visual>
         <origin xyz="0 0 0" rpy="0 0 0" />
@@ -29,8 +29,8 @@
       </inertial>
     </link>
-    <gazebo reference="camera_link">
+    <gazebo reference="${prefix}_camera_link">
         <material>Gazebo/Grey</material>
     </gazebo>
-    <gazebo reference="camera_link">
+    <gazebo reference="${prefix}_camera_link">
         <sensor type="camera" name="camera_node">
             <update_rate>30.0</update_rate>
@@ -55,8 +55,8 @@
                 <alwaysOn>true</alwaysOn>
                 <updateRate>0.0</updateRate>
-                <cameraName>/camera</cameraName>
+                <cameraName>/camera_${prefix}</cameraName>
                 <imageTopicName>image_raw</imageTopicName>
                 <cameraInfoTopicName>camera_info</cameraInfoTopicName>
-                <frameName>camera_link</frameName>
+                <frameName>${prefix}_camera_link</frameName>
                 <hackBaseline>0.07</hackBaseline>
                 <distortionK1>0.0</distortionK1>

File: robot_hunt_maze/urdf/sensor/laser.xacro (robot description, xacro)
@@ -1,4 +1,4 @@
 <?xml version="1.0" ?>
-<robot name="mbot" xmlns:xacro="http://www.ros.org/wiki/xacro">
+<robot name="laser" xmlns:xacro="http://www.ros.org/wiki/xacro">
   <xacro:macro name="laser" params="joint_x joint_y joint_z">
     <joint name="laser_joint" type="fixed">
